Commit message: fixed interval

File: arm1.urdf (robot description, URDF)
Before this commit: robot kicker-arm1, 6 links, 5 joints
Links:
- link player1: geometry collision box size=3 .5 5.5; visual box size=3 .5 5.5
- link player2: geometry collision box size=3 .5 5.5; visual box size=3 .5 5.5
- link player3: geometry collision box size=3 .5 5.5; visual box size=3 .5 5.5
- link rotator-link: geometry visual box size=10 10 10
- link slider-link: geometry visual box size=5 10 10
Joints:
- joint kernel-slider-joint: origin xyz=-0.60 0 0 rpy=0 0 0 -> xyz=-15 0 0 rpy=0 0 0
- joint player2-kernel-joint: origin xyz=-4.5 0 -0.75 rpy=0 0 0 -> xyz=-6 0 -0.75 rpy=0 0 0
- joint player3-kernel-joint: origin xyz=4.5 0 -0.75 rpy=0 0 0 -> xyz=6 0 -0.75 rpy=0 0 0
- joint slider-rotator-joint: origin xyz=-0.15 0 0 rpy=0 0 0 -> xyz=-7.5 0 0 rpy=0 0 0
