Commit message: board scene first look

File: models/board.urdf (robot description, URDF)
Before this commit: robot kicker-board, 9 links, 8 joints
Joints:
- joint bottom-left-board-joint: origin xyz=-7.25 7.25 2.5 rpy=0 0 0 -> xyz=-7.25 13.25 2.5 rpy=0 0 0
- joint bottom-right-board-joint: origin xyz=7.25 7.25 2.5 rpy=0 0 0 -> xyz=7.25 13.25 2.5 rpy=0 0 0
- joint top-left-board-joint: origin xyz=-7.25 -7.25 2.5 rpy=0 0 0 -> xyz=-7.25 -13.25 2.5 rpy=0 0 0
- joint top-right-board-joint: origin xyz=7.25 -7.25 2.5 rpy=0 0 0 -> xyz=7.25 -13.25 2.5 rpy=0 0 0
