Commit message: movement now works

File: models/arm1.urdf (robot description, URDF)
Before this commit: robot kicker-arm1, 6 links, 5 joints
Links:
- added link world
Joints:
- added joint rotator-world-joint: type fixed, parent world, child rotator-link
- joint slider-rotator-joint: limit lower=-3.14 upper=3.14 effort=10 velocity=3 -> lower=-1.57 upper=1.57 effort=10 velocity=3

File: models/arm2.urdf (robot description, URDF)
Before this commit: robot kicker-arm1, 6 links, 5 joints
Links:
- added link world
Joints:
- added joint rotator-world-joint: type fixed, parent world, child rotator-link

File: models/board.urdf (robot description, URDF)
Before this commit: robot kicker-board, 9 links, 8 joints
Links:
- added link world
Joints:
- added joint board-world-joint: type fixed, parent world, child board

Commit message: added movement on keydown

File: models/arm1.urdf (robot description, URDF)
Before this commit: robot kicker-arm1, 7 links, 6 joints
Links:
- link player1: geometry collision box size=3 .5 4; visual box size=3 .5 4
- link player2: geometry collision box size=3 .5 4; visual box size=3 .5 4
- link player3: geometry collision box size=3 .5 4; visual box size=3 .5 4

File: models/arm2.urdf (robot description, URDF)
Before this commit: robot kicker-arm1, 7 links, 6 joints
Links:
- link player1: geometry collision box size=3 .5 4; visual box size=3 .5 4
- link player2: geometry collision box size=3 .5 4; visual box size=3 .5 4
- link player3: geometry collision box size=3 .5 4; visual box size=3 .5 4
Joints:
- joint slider-rotator-joint: limit lower=-3.14 upper=3.14 effort=10 velocity=3 -> lower=-1.57 upper=1.57 effort=10 velocity=3
