Commit message: Fix players geometry

File: kicker/assets/arm1.urdf (robot description, URDF)
Before this commit: robot kicker-arm1, 7 links, 6 joints
Links:
- link player1: geometry collision box size=1.2 .5 4; visual box size=1.2 .5 4
- link player2: geometry collision box size=1.2 .5 4; visual box size=1.2 .5 4
- link player3: geometry collision box size=1.2 .5 4; visual box size=1.2 .5 4

File: kicker/assets/arm2.urdf (robot description, URDF)
Before this commit: robot kicker-arm1, 7 links, 6 joints
Links:
- link player1: geometry collision box size=1.2 .5 4; visual box size=1.2 .5 4
- link player2: geometry collision box size=1.2 .5 4; visual box size=1.2 .5 4
- link player3: geometry collision box size=1.2 .5 4; visual box size=1.2 .5 4
